Commit message: Tested for gazebo and ros_control.

File: yoyoman01_description/urdf/yoyoman01.xacro (robot description, xacro)
@@ -232,3 +232,68 @@
     </collision>
   </link>
+  <transmission name="tranHead">
+    <type>transmission_interface/SimpleTransmission</type>
+    <joint name="Head">
+      <hardwareInterface>hardware_interface/EffortJointInterface</hardwareInterface>
+    </joint>
+    <actuator name="motorHead">
+      <hardwareInterface>hardware_interface/EffortJointInterface</hardwareInterface>
+      <mechanicalReduction>1</mechanicalReduction>
+    </actuator>
+  </transmission>
+  <transmission name="tranNeck">
+    <type>transmission_interface/SimpleTransmission</type>
+    <joint name="Neck">
+      <hardwareInterface>hardware_interface/EffortJointInterface</hardwareInterface>
+    </joint>
+    <actuator name="motorNeck">
+      <hardwareInterface>hardware_interface/EffortJointInterface</hardwareInterface>
+      <mechanicalReduction>1</mechanicalReduction>
+    </actuator>
+  </transmission>
+  <transmission name="tranRarm">
+    <type>transmission_interface/SimpleTransmission</type>
+    <joint name="Rarm">
+      <hardwareInterface>hardware_interface/EffortJointInterface</hardwareInterface>
+    </joint>
+    <actuator name="motorRarm">
+      <hardwareInterface>hardware_interface/EffortJointInterface</hardwareInterface>
+      <mechanicalReduction>1</mechanicalReduction>
+    </actuator>
+  </transmission>
+  <transmission name="tranLarm">
+    <type>transmission_interface/SimpleTransmission</type>
+    <joint name="Larm">
+      <hardwareInterface>hardware_interface/EffortJointInterface</hardwareInterface>
+    </joint>
+    <actuator name="motorLarm">
+      <hardwareInterface>hardware_interface/EffortJointInterface</hardwareInterface>
+      <mechanicalReduction>1</mechanicalReduction>
+    </actuator>
+  </transmission>
+  <transmission name="tranRHip">
+    <type>transmission_interface/SimpleTransmission</type>
+    <joint name="RHip">
+      <hardwareInterface>hardware_interface/EffortJointInterface</hardwareInterface>
+    </joint>
+    <actuator name="motorRHip">
+      <hardwareInterface>hardware_interface/EffortJointInterface</hardwareInterface>
+      <mechanicalReduction>1</mechanicalReduction>
+    </actuator>
+  </transmission>
+  <transmission name="tranLHip">
+    <type>transmission_interface/SimpleTransmission</type>
+    <joint name="LHip">
+      <hardwareInterface>hardware_interface/EffortJointInterface</hardwareInterface>
+    </joint>
+    <actuator name="motorLHip">
+      <hardwareInterface>hardware_interface/EffortJointInterface</hardwareInterface>
+      <mechanicalReduction>1</mechanicalReduction>
+    </actuator>
+  </transmission>
+  <gazebo>
+    <plugin name="gazebo_ros_control" filename="libgazebo_ros_control.so">
+      <robotNamespace>/yoyoman01</robotNamespace>
+    </plugin>
+  </gazebo>
 </robot>

Commit message: MAJ modele urdf

File: yoyoman01_description/urdf/yoyoman01.xacro (robot description, xacro)
@@ -14,10 +14,10 @@
     <parent link="world"/>
     <child link="base_link"/>
-  </joint>
+</joint>
   <link name="base_link">
     <inertial>
-      <mass value="0.663"/>
-      <inertia ixx="0.049" ixy="-3.058e-7" ixz="-0.00004029" iyy="0.043" iyz="1.539e-5" izz="0.006"/>
-      <origin rpy="0 0 0" xyz="0 0 0.388"/>
+      <mass value="1.635"/>
+      <inertia ixx="86e-03" ixy="-39.84e-6" ixz="3.991e-4" iyy="83e-3" iyz="-38.29e-6" izz="4e-3"/>
+      <origin rpy="0 0 0" xyz="0 0 0.17346"/>
     </inertial>
     <visual>
@@ -25,4 +25,5 @@
         <mesh filename="package://yoyoman01_description/meshes/BUSTE.stl" scale="0.001 0.001 0.001"/>
       </geometry>
+    <origin rpy="0 0 -1.57075" xyz="0 0 0"/>
     <material name="blue"/>
     </visual>
@@ -30,4 +31,29 @@
       <geometry>
         <mesh filename="package://yoyoman01_description/meshes/BUSTE.stl" scale="0.001 0.001 0.001"/>
+      </geometry>
+    </collision>
+  </link>
+  <joint name="Neck" type="revolute">
+    <parent link="base_link"/>
+    <child link="NeckLink"/>
+    <origin rpy="0 0 0" xyz="0 0 0.675"/>
+    <axis xyz="0 1 0"/>
+    <limit effort="0.5" lower="0" upper="0.5" velocity="1"/>
+  </joint>
+  <link name="NeckLink">
+    <inertial>
+      <mass value="0.061"/>
+      <inertia ixx="2.95e-5" ixy="-7.67e-9" ixz="-3.61e-9" iyy="2.53e-5" iyz="-3.05e-6" izz="1.09e-5"/>
+      <origin rpy="0 0 0" xyz="0 0 0.03"/>
+    </inertial>
+    <visual>
+      <geometry>
+        <mesh filename="package://yoyoman01_description/meshes/COU.stl" scale="0.001 0.001 0.001"/>
+      </geometry>
+    <origin rpy="0 0 1.57075" xyz="0 0 0"/>
+    </visual>
+    <collision>
+      <geometry>
+        <mesh filename="package://yoyoman01_description/meshes/COU.stl" scale="0.001 0.001 0.001"/>
       </geometry>
     </collision>
@@ -36,13 +62,13 @@
     <parent link="NeckLink"/>
     <child link="HeadLink"/>
-    <origin rpy="0 0 0" xyz="0 0 0.056"/>
-    <axis xyz="0 1.0 0"/>
+    <origin rpy="0 0 0" xyz="0 0 0.064502"/>
+    <axis xyz="0 1 0"/>
     <limit effort="0.5" lower="0" upper="0.5" velocity="1"/>
   </joint>
   <link name="HeadLink">
     <inertial>
-      <mass value="0.254"/>
-      <inertia ixx="0.003" ixy="0.00" ixz="-5.71E-008" iyy="0.001" iyz="0.00" izz="0.001"/>
-      <origin rpy="0 0 0" xyz="0 0 0.1"/>
+      <mass value="0.340"/>
+      <inertia ixx="2e-3" ixy="-129.7e-9" ixz="5.391e-5" iyy="3e-3" iyz="-267.9e-9" izz="1e-3"/>
+      <origin rpy="0 0 0" xyz="0 0 0.143385"/>
     </inertial>
     <visual>
@@ -50,5 +76,5 @@
         <mesh filename="package://yoyoman01_description/meshes/TETE.stl" scale="0.001 0.001 0.001"/>
       </geometry>
-    <origin rpy="0 0 0 " xyz="0 0 0"/>
+    <origin rpy="0 0 1.57075 " xyz="0 0 0"/>
     <material name="blue"/>
     </visual>
@@ -59,40 +85,16 @@
     </collision>
   </link>
-  <joint name="Neck" type="revolute">
-    <parent link="base_link"/>
-    <child link="NeckLink"/>
-    <origin rpy="0 0 0" xyz="0 0 0.669"/>
-    <axis xyz="0 1.0 0"/>
-    <limit effort="0.5" lower="0" upper="0.5" velocity="1"/>
-  </joint>
-  <link name="NeckLink">
-    <inertial>
-      <mass value="0.061"/>
-      <inertia ixx="2.791e-5" ixy="6.564e-10" ixz="-0.000000001" iyy="2.334e-5" iyz="8.312e-7" izz="1.155e-5"/>
-      <origin rpy="0 0 0" xyz="0 0 0.03"/>
-    </inertial>
-    <visual>
-      <geometry>
-        <mesh filename="package://yoyoman01_description/meshes/COU.stl" scale="0.001 0.001 0.001"/>
-      </geometry>
-    </visual>
-    <collision>
-      <geometry>
-        <mesh filename="package://yoyoman01_description/meshes/COU.stl" scale="0.001 0.001 0.001"/>
-      </geometry>
-    </collision>
-  </link>
 <joint name="Rarm" type="revolute">
     <parent link="base_link"/>
     <child link="RArmLink"/>
-    <origin rpy="0 0 0" xyz="0 -0.155 0.580 "/>
-    <axis xyz="0 1.0 0"/>
+    <origin rpy="0 0 0" xyz="0 -0.155 0.589901 "/>
+    <axis xyz="0 1 0"/>
     <limit effort="5" lower="0" upper="5" velocity="1"/>
   </joint>
 <link name="RArmLink">
     <inertial>
-      <mass value="0.237"/>
-      <inertia ixx="0.002" ixy="2.19e-20" ixz="7.418e-20" iyy="0.002" iyz="1.207e-6" izz="6.001e-5"/>
-      <origin rpy="0 0 0 " xyz="0 0 -0.322"/>
+      <mass value="0.172"/>
+      <inertia ixx="3e-3" ixy="-2.011e-20" ixz="-3.61e-9" iyy="3e-3" iyz="3.05e-6" izz="2.475e-5"/>
+      <origin rpy="0 0 0 " xyz="0 0 -0.10032"/>
     </inertial>
     <visual>
@@ -100,5 +102,5 @@
         <mesh filename="package://yoyoman01_description/meshes/BRAS.stl" scale="0.001 0.001 0.001"/>
       </geometry>
-    <origin rpy="0 0 3.14" xyz="0 0 0"/>
+    <origin rpy="0 0 -1.57075" xyz="0 0 0"/>
     </visual>
     <collision>
@@ -111,13 +113,13 @@
     <parent link="base_link"/>
     <child link="LArmLink"/>
-    <origin rpy="0 0 0" xyz="0 0.155 0.580 "/>
-    <axis xyz="0 1.0 0"/>
+    <origin rpy="0 0 0" xyz="0 0.155 0.589901 "/>
+    <axis xyz="0 1 0"/>
     <limit effort="2.57" lower="-0.349066" upper="0.279253" velocity="1.9"/>
   </joint>
 <link name="LArmLink">
     <inertial>
-      <mass value="0.237"/>
-      <inertia ixx="0.002" ixy="-2.19e-20" ixz="7.418e-20" iyy="0.002" iyz="-1.207e-6" izz="6.001e-5"/>
-      <origin rpy="0 0 0" xyz="0 0 -0.322"/>
+      <mass value="0.172"/>
+      <inertia ixx="3e-3" ixy="2.011e-20" ixz="-3.61e-9" iyy="3e-3" iyz="-3.05e-6" izz="2.475e-5"/>
+      <origin rpy="0 0 0 " xyz="0 0 -0.10032"/>
     </inertial>
     <visual>
@@ -125,5 +127,5 @@
         <mesh filename="package://yoyoman01_description/meshes/BRAS.stl" scale="0.001 0.001 0.001"/>
       </geometry>
-    <origin rpy="0 0 0" xyz="0 0 0"/>
+    <origin rpy="0 0 1.57075" xyz="0 0 0"/>
     </visual>
     <collision>
@@ -142,7 +144,7 @@
   <link name="RHipLink">
     <inertial>
-      <mass value="0.92"/>
+      <mass value="0.816"/>
       <inertia ixx="0.001" ixy="1.921e-4" ixz="-0.0001443" iyy="0.002" iyz="1.291e-4" izz="0.002"/>
-      <origin rpy="0 0 0" xyz="0.038 -0.034 0.007"/>
+      <origin rpy="0 0 0" xyz="0.0506 -0.0137 0.0101"/>
     </inertial>
     <visual>
@@ -150,4 +152,5 @@
         <mesh filename="package://yoyoman01_description/meshes/HANCHE_D.stl" scale="0.001 0.001 0.001"/>
       </geometry>
+    <origin rpy="0 3.14 1.57075" xyz="0 0 0"/>
     </visual>
     <collision>
@@ -166,7 +169,7 @@
   <link name="LHipLink">
     <inertial>
-      <mass value="0.92"/>
+      <mass value="0.816"/>
       <inertia ixx="0.001" ixy="-1.921e-4" ixz="-0.0001443" iyy="0.002" iyz="-1.291e-4" izz="0.002"/>
-      <origin rpy="0 0 0" xyz="0.038 0.034 0.007"/>
+      <origin rpy="0 0 0" xyz="0.0506 0.0137 0.0101"/>
     </inertial>
     <visual>
@@ -174,4 +177,5 @@
         <mesh filename="package://yoyoman01_description/meshes/HANCHE_G.stl" scale="0.001 0.001 0.001"/>
       </geometry>
+    <origin rpy="0 0 1.57075" xyz="0 0 0"/>
     </visual>
     <collision>
@@ -184,23 +188,24 @@
     <parent link="RHipLink"/>
     <child link="RKneeLink"/>
-    <origin rpy="0 0 0" xyz="0.015 -0.068 -0.04"/>
-    <axis xyz="0 0 1"/>
+    <origin rpy="0 0 0" xyz="-0.021 -0.068 -0.01"/>
+    <axis xyz="0 0 0"/>
     <limit effort="50" lower="0" upper="0.04" velocity="1"/>
   </joint>
   <link name="RKneeLink">
     <inertial>
-      <mass value="0.527"/>
-      <inertia ixx="0.052" ixy="1.464e-5" ixz="-0.00006891" iyy="0.052" iyz="0.002" izz="0.001"/>
-      <origin rpy="0 0 0" xyz="0.002 0.017 -0.560"/>
-    </inertial>
-    <visual>
-      <geometry>
-        <mesh filename="package://yoyoman01_description/meshes/JAMBE_D.stl" scale="0.001 0.001 0.001"/>
-      </geometry>
+      <mass value="0.839"/>
+      <inertia ixx="80e-3" ixy="17.42e-6" ixz="-154.3e-6" iyy="80e-3" iyz="-3e-3" izz="2e-3"/>
+      <origin rpy="0 0 0" xyz="0.01817 -0.01317 -0.557"/>
+    </inertial>
+    <visual>
+      <geometry>
+        <mesh filename="package://yoyoman01_description/meshes/JAMBE_G.stl" scale="0.001 0.001 0.001"/>
+      </geometry>
+    <origin rpy="0 0 3.14" xyz="0 0 0"/>
     <material name="blue"/>
     </visual>
     <collision>
       <geometry>
-        <mesh filename="package://yoyoman01_description/meshes/JAMBE_D.stl" scale="0.001 0.001 0.001"/>
+        <mesh filename="package://yoyoman01_description/meshes/JAMBE_G.stl" scale="0.001 0.001 0.001"/>
       </geometry>
     </collision>
@@ -209,17 +214,17 @@
     <parent link="LHipLink"/>
     <child link="LKneeLink"/>
-    <origin rpy="0 0 0" xyz="0.015 0.068 -0.04"/>
-    <axis xyz="0 0 1"/>
+    <origin rpy="0 0 0" xyz="-0.021 0.068 -0.01"/>
+    <axis xyz="0 0 0"/>
     <limit effort="50" lower="0" upper="0.04" velocity="1"/>
   </joint>
   <link name="LKneeLink">
     <inertial>
-      <mass value="0.527"/>
-      <inertia ixx="0.052" ixy="-1.464e-5" ixz="-0.00006891" iyy="0.052" iyz="-0.002" izz="0.001"/>
-      <origin rpy="0 0 0" xyz="0.002 -0.017 -0.560"/>
-    </inertial>
-    <visual>
-      <geometry>
-        <mesh filename="package://yoyoman01_description/meshes/JAMBE_G.stl" scale="0.001 0.001 0.001"/>
+      <mass value="0.839"/>
+      <inertia ixx="80e-3" ixy="-17.42e-6" ixz="-154.3e-6" iyy="80e-3" iyz="3e-3" izz="2e-3"/>
+      <origin rpy="0 0 0" xyz="0.01817 0.01317 -0.557"/>
+    </inertial>
+    <visual>
+      <geometry>
+        <mesh filename="package://yoyoman01_description/meshes/JAMBE_D.stl" scale="0.001 0.001 0.001"/>
       </geometry>
     <origin rpy="0 0 3.14" xyz="0 0 0"/>
@@ -228,8 +233,11 @@
     <collision>
       <geometry>
-        <mesh filename="package://yoyoman01_description/meshes/JAMBE_G.stl" scale="0.001 0.001 0.001"/>
-      </geometry>
-    </collision>
-  </link>
+        <mesh filename="package://yoyoman01_description/meshes/JAMBE_D.stl" scale="0.001 0.001 0.001"/>
+      </geometry>
+    </collision>
+  </link>
+<!--
+**********Transmissions**********
+-->
   <transmission name="tranHead">
     <type>transmission_interface/SimpleTransmission</type>

Commit message: ajout points de reference pieds

File: yoyoman01_description/urdf/yoyoman01.xacro (robot description, xacro)
@@ -237,4 +237,21 @@
     </collision>
   </link>
+<!-- **********Virtual points on the top of the foots ********** -->
+  <joint name="RFoot" type="fixed">
+    <parent link="RKneeLink"/>
+    <child link="RFootLink"/>
+    <origin rpy="0 0 0" xyz="-0.0187 0 -0.7775"/>
+    <axis xyz="0 0 0"/>
+  </joint>
+    <link name="RFootLink">
+  </link>link>
+  <joint name="LFoot" type="fixed">
+    <parent link="LKneeLink"/>
+    <child link="LFootLink"/>
+    <origin rpy="0 0 0" xyz="-0.0187 0 -0.7775"/>
+    <axis xyz="0 0 0"/>
+  </joint>
+    <link name="LFootLink">
+  </link>link>
 <!--
 **********Transmissions**********

Commit message: fixing collision model

File: yoyoman01_description/urdf/yoyoman01.xacro (robot description, xacro)
@@ -19,5 +19,5 @@
       <mass value="1.635"/>
       <inertia ixx="86e-03" ixy="-39.84e-6" ixz="3.991e-4" iyy="83e-3" iyz="-38.29e-6" izz="4e-3"/>
-      <origin rpy="0 0 0" xyz="0 0 0.17346"/>
+      <origin rpy="0 0 -1.57075" xyz="0 0 0.17346"/>
     </inertial>
     <visual>
@@ -25,7 +25,9 @@
         <mesh filename="package://yoyoman01_description/meshes/BUSTE.stl" scale="0.001 0.001 0.001"/>
       </geometry>
+    <material name="blue"/>
+    </visual>
+<!--
     <origin rpy="0 0 -1.57075" xyz="0 0 0"/>
-    <material name="blue"/>
-    </visual>
+-->
     <collision>
       <geometry>

Commit message: fixing collision model

File: yoyoman01_description/urdf/yoyoman01.xacro (robot description, xacro)
@@ -19,5 +19,5 @@
       <mass value="1.635"/>
       <inertia ixx="86e-03" ixy="-39.84e-6" ixz="3.991e-4" iyy="83e-3" iyz="-38.29e-6" izz="4e-3"/>
-      <origin rpy="0 0 -1.57075" xyz="0 0 0.17346"/>
+      <origin rpy="0 0 0" xyz="0 0 0.17346"/>
     </inertial>
     <visual>
@@ -25,13 +25,12 @@
         <mesh filename="package://yoyoman01_description/meshes/BUSTE.stl" scale="0.001 0.001 0.001"/>
       </geometry>
+    <origin rpy="0 0 -1.57075" xyz="0 0 0"/>
     <material name="blue"/>
     </visual>
-<!--
+    <collision>
+      <geometry>
+        <mesh filename="package://yoyoman01_description/meshes/BUSTE.stl" scale="0.001 0.001 0.001"/>
+      </geometry>
     <origin rpy="0 0 -1.57075" xyz="0 0 0"/>
--->
-    <collision>
-      <geometry>
-        <mesh filename="package://yoyoman01_description/meshes/BUSTE.stl" scale="0.001 0.001 0.001"/>
-      </geometry>
     </collision>
   </link>
@@ -59,4 +58,5 @@
         <mesh filename="package://yoyoman01_description/meshes/COU.stl" scale="0.001 0.001 0.001"/>
       </geometry>
+    <origin rpy="0 0 1.57075" xyz="0 0 0"/>
     </collision>
   </link>
@@ -85,4 +85,5 @@
         <mesh filename="package://yoyoman01_description/meshes/TETE.stl" scale="0.001 0.001 0.001"/>
       </geometry>
+    <origin rpy="0 0 1.57075 " xyz="0 0 0"/>
     </collision>
   </link>
@@ -110,4 +111,5 @@
         <mesh filename="package://yoyoman01_description/meshes/BRAS.stl" scale="0.001 0.001 0.001"/>
       </geometry>
+    <origin rpy="0 0 -1.57075" xyz="0 0 0"/>
     </collision>
   </link>
@@ -135,4 +137,5 @@
         <mesh filename="package://yoyoman01_description/meshes/BRAS.stl" scale="0.001 0.001 0.001"/>
       </geometry>
+    <origin rpy="0 0 1.57075" xyz="0 0 0"/>
     </collision>
   </link>
@@ -160,4 +163,5 @@
         <mesh filename="package://yoyoman01_description/meshes/HANCHE_D.stl" scale="0.001 0.001 0.001"/>
       </geometry>
+    <origin rpy="0 3.14 1.57075" xyz="0 0 0"/>
     </collision>
   </link>
@@ -185,4 +189,5 @@
         <mesh filename="package://yoyoman01_description/meshes/HANCHE_G.stl" scale="0.001 0.001 0.001"/>
       </geometry>
+    <origin rpy="0 0 1.57075" xyz="0 0 0"/>
     </collision>
   </link>
@@ -211,4 +216,5 @@
         <mesh filename="package://yoyoman01_description/meshes/JAMBE_G.stl" scale="0.001 0.001 0.001"/>
       </geometry>
+    <origin rpy="0 0 3.14" xyz="0 0 0"/>
     </collision>
   </link>
@@ -237,4 +243,5 @@
         <mesh filename="package://yoyoman01_description/meshes/JAMBE_D.stl" scale="0.001 0.001 0.001"/>
       </geometry>
+    <origin rpy="0 0 3.14" xyz="0 0 0"/>
     </collision>
   </link>

Commit message: fixing x origin on RFoot and LFoot

File: yoyoman01_description/urdf/yoyoman01.xacro (robot description, xacro)
@@ -250,17 +250,17 @@
     <parent link="RKneeLink"/>
     <child link="RFootLink"/>
-    <origin rpy="0 0 0" xyz="-0.0187 0 -0.7775"/>
+    <origin rpy="0 0 0" xyz="0.0187 0 -0.7775"/>
     <axis xyz="0 0 0"/>
   </joint>
     <link name="RFootLink">
-  </link>link>
+  </link>
   <joint name="LFoot" type="fixed">
     <parent link="LKneeLink"/>
     <child link="LFootLink"/>
-    <origin rpy="0 0 0" xyz="-0.0187 0 -0.7775"/>
+    <origin rpy="0 0 0" xyz="0.0187 0 -0.7775"/>
     <axis xyz="0 0 0"/>
   </joint>
     <link name="LFootLink">
-  </link>link>
+  </link>
 <!--
 **********Transmissions**********
