Commit message: Add files via upload

File: yoyoman01_traject/urdf/barriere.xacro (robot description, xacro)
@@ -19,21 +19,11 @@
         <mesh filename="package://yoyoman01_description/meshes/barre600.stl" scale="0.001 0.001 0.001"/>
       </geometry>
-    <origin rpy="0 0 0" xyz="-0.3 0 0"/>
+    <origin rpy="0 0 0" xyz="-0.5 0 0"/>
     </visual>
     <collision>
-      <selfCollide>true</selfCollide>
       <geometry>
         <mesh filename="package://yoyoman01_description/meshes/barre.stl" scale="0.001 0.001 0.001"/>
       </geometry>
-    <origin rpy="0 0 0" xyz="-0.3 0 0"/>
+    <origin rpy="0 0 0" xyz="-0.5 0 0"/>
     </collision>
   </link>
-  <gazebo>
-    <plugin name="gazebo_ros_control" filename="libgazebo_ros_control.so">
-      <!--robotNamespace>/yoyoman01</robotNamespace-->
-    </plugin>
-    <selfCollide>true</selfCollide>
-    <static>false</static>
-    <turnGravityOff>false</turnGravityOff>
-  </gazebo>
-</robot>

File: yoyoman01_traject/urdf/yoyoman01.xacro (robot description, xacro)
@@ -10,9 +10,9 @@
       <color rgba="0 0 0.8 1"/>
    </material>
-   <link name="world"/>
+   <!--link name="world"/>
   <joint name="fixed" type="fixed">
     <parent link="world"/>
     <child link="base_link"/>
-</joint>
+</joint-->
   <link name="base_link">
     <inertial>
@@ -40,5 +40,5 @@
     <origin rpy="0 0 0" xyz="0 0 0.675"/>
     <axis xyz="0 1 0"/>
-    <limit effort="0.5" lower="0" upper="0.5" velocity="1"/>
+    <limit effort="10.5" lower="-0.5" upper="0.5" velocity="1"/>
   </joint>
   <link name="NeckLink">
@@ -66,5 +66,5 @@
     <origin rpy="0 0 0" xyz="0 0 0.064502"/>
     <axis xyz="0 1 0"/>
-    <limit effort="0.5" lower="0" upper="0.5" velocity="1"/>
+    <limit effort="10.5" lower="-0.5" upper="0.5" velocity="1"/>
   </joint>
   <link name="HeadLink">
@@ -93,5 +93,5 @@
     <origin rpy="0 0 0" xyz="0 -0.155 0.589901 "/>
     <axis xyz="0 1 0"/>
-    <limit effort="5" lower="0" upper="5" velocity="1"/>
+    <limit effort="50" lower="-3" upper="3" velocity="10"/>
   </joint>
 <link name="RArmLink">
@@ -119,5 +119,5 @@
     <origin rpy="0 0 0" xyz="0 0.155 0.589901 "/>
     <axis xyz="0 1 0"/>
-    <limit effort="2.57" lower="-0.349066" upper="0.279253" velocity="1.9"/>
+    <limit effort="50" lower="-3" upper="3" velocity="10"/>
   </joint>
 <link name="LArmLink">
@@ -145,5 +145,5 @@
     <origin rpy="0 0 0" xyz="0 -0.09 0"/>
     <axis xyz="0 1 0"/>
-    <limit effort="6" lower="0" upper="6" velocity="1"/>
+    <limit effort="600" lower="-3" upper="3" velocity="10"/>
   </joint>
   <link name="RHipLink">
@@ -171,5 +171,5 @@
     <origin rpy="0 0 0" xyz="0 0.09 0"/>
     <axis xyz="0 1 0"/>
-    <limit effort="6" lower="0" upper="6" velocity="1"/>
+    <limit effort="600" lower="-3" upper="3" velocity="10"/>
   </joint>
   <link name="LHipLink">
@@ -330,4 +330,5 @@
       <!--robotNamespace>/yoyoman01</robotNamespace-->
     </plugin>
+    <selfCollide>true</selfCollide>
   </gazebo>
 </robot>
