Commit message: Add files via upload

File: yoyoman01_traject/urdf/yoyoman01.xacro (robot description, xacro)
@@ -34,4 +34,5 @@
     <origin rpy="0 0 -1.57075" xyz="0 0 0"/>
     </collision>
+  <velocity rpy="0 0 0" xyz="10 10 10000000000000000000000000000000000000000000000000000000000"/>
   </link>
   <joint name="Neck" type="revolute">
@@ -40,5 +41,5 @@
     <origin rpy="0 0 0" xyz="0 0 0.675"/>
     <axis xyz="0 1 0"/>
-    <limit effort="10.5" lower="-0.5" upper="0.5" velocity="1"/>
+    <limit effort="1.5" lower="-0.5" upper="0.5" velocity="6.175333333"/>
   </joint>
   <link name="NeckLink">
@@ -66,5 +67,5 @@
     <origin rpy="0 0 0" xyz="0 0 0.064502"/>
     <axis xyz="0 1 0"/>
-    <limit effort="10.5" lower="-0.5" upper="0.5" velocity="1"/>
+    <limit effort="1.5" lower="-0.5" upper="0.5" velocity="6.175333333"/>
   </joint>
   <link name="HeadLink">
@@ -93,5 +94,5 @@
     <origin rpy="0 0 0" xyz="0 -0.155 0.589901 "/>
     <axis xyz="0 1 0"/>
-    <limit effort="50" lower="-3" upper="3" velocity="10"/>
+    <limit effort="4.1" lower="-3" upper="3" velocity="4.81"/>
   </joint>
 <link name="RArmLink">
@@ -119,5 +120,5 @@
     <origin rpy="0 0 0" xyz="0 0.155 0.589901 "/>
     <axis xyz="0 1 0"/>
-    <limit effort="50" lower="-3" upper="3" velocity="10"/>
+    <limit effort="4.1" lower="-3" upper="3" velocity="4.814666667"/>
   </joint>
 <link name="LArmLink">
@@ -145,5 +146,5 @@
     <origin rpy="0 0 0" xyz="0 -0.09 0"/>
     <axis xyz="0 1 0"/>
-    <limit effort="600" lower="-3" upper="3" velocity="10"/>
+    <limit effort="6.672" lower="-3" upper="19.079861111" velocity="10"/>
   </joint>
   <link name="RHipLink">
@@ -171,5 +172,5 @@
     <origin rpy="0 0 0" xyz="0 0.09 0"/>
     <axis xyz="0 1 0"/>
-    <limit effort="600" lower="-3" upper="3" velocity="10"/>
+    <limit effort="4.1" lower="-3" upper="3" velocity="4.814666667"/>
   </joint>
   <link name="LHipLink">

Commit message: Add files via upload

File: yoyoman01_traject/urdf/yoyoman01.xacro (robot description, xacro)
@@ -264,4 +264,31 @@
     <link name="LFootLink">
   </link>
+<!-- IMU -->
+<link name="imu_link">
+  <inertial>
+    <mass value="0.00"/>
+    <origin rpy="0 0 0" xyz="0 0 0"/>
+    <inertia ixx="0.000" ixy="0" ixz="0" iyy="0.000" iyz="0" izz="0.000"/>
+  </inertial>
+  <visual>
+    <origin rpy="0 0 0" xyz="0 0 0"/>
+    <geometry>
+      <sphere radius="0.01"/>
+    </geometry>
+  </visual>
+  <collision>
+    <origin rpy="0 0 0" xyz="0 0 0"/>
+    <geometry>
+      <sphere radius="0.01"/>
+    </geometry>
+  </collision>
+</link>
+<!-- IMU Joint -->
+  <joint name="imu_joint" type="fixed">
+    <axis xyz="0 0 0"/> <!-- 0 1 0 -->
+    <origin xyz="0 0 0.15"/>
+    <parent link="HeadLink"/>
+    <child link="imu_link"/>
+  </joint>
 <!--
 **********Transmissions**********
@@ -327,9 +354,32 @@
     </actuator>
   </transmission>
-  <gazebo>
+<gazebo>
     <plugin name="gazebo_ros_control" filename="libgazebo_ros_control.so">
       <!--robotNamespace>/yoyoman01</robotNamespace-->
     </plugin>
     <selfCollide>true</selfCollide>
+<!-- IMU-->
+      <plugin name="imu_plugin" filename="libhector_gazebo_ros_imu.so">
+            <alwaysOn>true</alwaysOn>
+            <updateRate>1000</updateRate>
+            <bodyName>imu_link</bodyName>
+            <topicName>/imu</topicName>
+            <serviceName>/imu/calibrate</serviceName>
+            <accelOffset>0.0 0.0 0.0</accelOffset>
+            <accelDrift>0.0 0.0 0.0</accelDrift>
+            <accelDriftFrequency>0.0 0.0 0.0</accelDriftFrequency>
+            <accelGaussianNoise>0.0 0.0 0.0</accelGaussianNoise>
+            <rateOffset>0.0 0.0 0.0</rateOffset>
+            <rateDrift>0.0 0.0 0.0</rateDrift>
+            <rateDriftFrequency>0.0 0.0 0.0</rateDriftFrequency>
+            <rateGaussianNoise>0.0 0.0 0.0</rateGaussianNoise>
+            <headingOffset>0.0</headingOffset>
+            <headingDrift>0.0</headingDrift>
+            <headingDriftFrequency>0.0</headingDriftFrequency>
+            <headingGaussianNoise>0.0</headingGaussianNoise>
+            <rpyOffset>0.0 0.0 0.0</rpyOffset>
+            <xyzOffset>0.0 0.0 0.0</xyzOffset>
+            <gaussianNoise>0.0</gaussianNoise>
+        </plugin>
   </gazebo>
 </robot>

Commit message: Add files via upload

File: yoyoman01_traject/urdf/yoyoman01.xacro (robot description, xacro)
@@ -15,4 +15,10 @@
     <child link="base_link"/>
 </joint-->
+<!-- virtual link with a virtual joint to make the root link -->
+  <link name="virtual_link"/>
+  <joint name="virtual_joint" type="fixed">
+    <parent link="virtual_link"/>
+    <child link="base_link"/>
+  </joint>
   <link name="base_link">
     <inertial>
@@ -34,5 +40,4 @@
     <origin rpy="0 0 -1.57075" xyz="0 0 0"/>
     </collision>
-  <velocity rpy="0 0 0" xyz="10 10 10000000000000000000000000000000000000000000000000000000000"/>
   </link>
   <joint name="Neck" type="revolute">
@@ -383,3 +388,25 @@
         </plugin>
   </gazebo>
+  <gazebo reference="imu_link">
+    <plugin name="gazebo_ros_control" filename="libgazebo_ros_control.so">
+    </plugin>
+    <selfCollide>true</selfCollide>
+    <gravity>true</gravity>
+    <sensor name="imu_sensor" type="imu">
+      <always_on>true</always_on>
+      <update_rate>100</update_rate>
+      <visualize>true</visualize>
+      <topic>__default_topic__</topic>
+      <plugin filename="libgazebo_ros_imu_sensor.so" name="imu_plugin">
+        <topicName>imu</topicName>
+        <bodyName>imu_link</bodyName>
+        <updateRateHZ>1000.0</updateRateHZ>
+        <gaussianNoise>0.0</gaussianNoise>
+        <xyzOffset>0 0 0</xyzOffset>
+        <rpyOffset>0 0 0</rpyOffset>
+        <frameName>imu_link</frameName>
+      </plugin>
+      <pose>0 0 0 0 0 0</pose>
+    </sensor>
+  </gazebo>
 </robot>

Commit message: Add files via upload

File: yoyoman01_traject/urdf/yoyoman01.xacro (robot description, xacro)
@@ -10,15 +10,15 @@
       <color rgba="0 0 0.8 1"/>
    </material>
-   <!--link name="world"/>
+   <link name="world"/>
   <joint name="fixed" type="fixed">
     <parent link="world"/>
     <child link="base_link"/>
-</joint-->
+</joint>
 <!-- virtual link with a virtual joint to make the root link -->
-  <link name="virtual_link"/>
+  <!--link name="virtual_link"/>
   <joint name="virtual_joint" type="fixed">
     <parent link="virtual_link"/>
     <child link="base_link"/>
-  </joint>
+  </joint-->
   <link name="base_link">
     <inertial>
@@ -367,5 +367,5 @@
       <plugin name="imu_plugin" filename="libhector_gazebo_ros_imu.so">
             <alwaysOn>true</alwaysOn>
-            <updateRate>1000</updateRate>
+            <updateRate>10</updateRate>
             <bodyName>imu_link</bodyName>
             <topicName>/imu</topicName>
@@ -395,5 +395,5 @@
     <sensor name="imu_sensor" type="imu">
       <always_on>true</always_on>
-      <update_rate>100</update_rate>
+      <update_rate>1000.0</update_rate>
       <visualize>true</visualize>
       <topic>__default_topic__</topic>

Commit message: adding yoyoman01.update and connection to rviz

File: yoyoman01_traject/urdf/yoyoman01.xacro (robot description, xacro)
@@ -46,5 +46,5 @@
     <origin rpy="0 0 0" xyz="0 0 0.675"/>
     <axis xyz="0 1 0"/>
-    <limit effort="1.5" lower="-0.5" upper="0.5" velocity="6.175333333"/>
+    <limit effort="1.5" lower="-2" upper="2" velocity="6.175333333"/>
   </joint>
   <link name="NeckLink">
@@ -72,5 +72,5 @@
     <origin rpy="0 0 0" xyz="0 0 0.064502"/>
     <axis xyz="0 1 0"/>
-    <limit effort="1.5" lower="-0.5" upper="0.5" velocity="6.175333333"/>
+    <limit effort="1.5" lower="-2" upper="2" velocity="6.175333333"/>
   </joint>
   <link name="HeadLink">

Commit message: fixing gravity issue passing to velocity interface

File: yoyoman01_traject/urdf/yoyoman01.xacro (robot description, xacro)
@@ -10,12 +10,12 @@
       <color rgba="0 0 0.8 1"/>
    </material>
-   <link name="world"/>
-  <joint name="fixed" type="fixed">
+   <!--link name="world"/>
+  <joint name="fixed" type="floating">
     <parent link="world"/>
     <child link="base_link"/>
-</joint>
-<!-- virtual link with a virtual joint to make the root link -->
+    </joint-->
+<!-- virtual link with a virtual joint to make the root link-->
   <!--link name="virtual_link"/>
-  <joint name="virtual_joint" type="fixed">
+  <joint name="virtual_joint" type="floating">
     <parent link="virtual_link"/>
     <child link="base_link"/>
@@ -302,8 +302,8 @@
     <type>transmission_interface/SimpleTransmission</type>
     <joint name="Head">
-      <hardwareInterface>hardware_interface/PositionJointInterface</hardwareInterface>
+      <hardwareInterface>hardware_interface/VelocityJointInterface</hardwareInterface>
     </joint>
     <actuator name="motorHead">
-      <hardwareInterface>hardware_interface/PositionJointInterface</hardwareInterface>
+      <hardwareInterface>hardware_interface/VelocityJointInterface</hardwareInterface>
       <mechanicalReduction>1</mechanicalReduction>
     </actuator>
@@ -312,8 +312,8 @@
     <type>transmission_interface/SimpleTransmission</type>
     <joint name="Neck">
-      <hardwareInterface>hardware_interface/PositionJointInterface</hardwareInterface>
+      <hardwareInterface>hardware_interface/VelocityJointInterface</hardwareInterface>
     </joint>
     <actuator name="motorNeck">
-      <hardwareInterface>hardware_interface/PositionJointInterface</hardwareInterface>
+      <hardwareInterface>hardware_interface/VelocityJointInterface</hardwareInterface>
       <mechanicalReduction>1</mechanicalReduction>
     </actuator>
@@ -322,8 +322,8 @@
     <type>transmission_interface/SimpleTransmission</type>
     <joint name="Rarm">
-      <hardwareInterface>hardware_interface/PositionJointInterface</hardwareInterface>
+      <hardwareInterface>hardware_interface/VelocityJointInterface</hardwareInterface>
     </joint>
     <actuator name="motorRarm">
-      <hardwareInterface>hardware_interface/PositionJointInterface</hardwareInterface>
+      <hardwareInterface>hardware_interface/VelocityJointInterface</hardwareInterface>
       <mechanicalReduction>1</mechanicalReduction>
     </actuator>
@@ -332,8 +332,8 @@
     <type>transmission_interface/SimpleTransmission</type>
     <joint name="Larm">
-      <hardwareInterface>hardware_interface/PositionJointInterface</hardwareInterface>
+      <hardwareInterface>hardware_interface/VelocityJointInterface</hardwareInterface>
     </joint>
     <actuator name="motorLarm">
-      <hardwareInterface>hardware_interface/PositionJointInterface</hardwareInterface>
+      <hardwareInterface>hardware_interface/VelocityJointInterface</hardwareInterface>
       <mechanicalReduction>1</mechanicalReduction>
     </actuator>
@@ -342,8 +342,8 @@
     <type>transmission_interface/SimpleTransmission</type>
     <joint name="RHip">
-      <hardwareInterface>hardware_interface/PositionJointInterface</hardwareInterface>
+      <hardwareInterface>hardware_interface/VelocityJointInterface</hardwareInterface>
     </joint>
     <actuator name="motorRHip">
-      <hardwareInterface>hardware_interface/PositionJointInterface</hardwareInterface>
+      <hardwareInterface>hardware_interface/VelocityJointInterface</hardwareInterface>
       <mechanicalReduction>1</mechanicalReduction>
     </actuator>
@@ -352,8 +352,8 @@
     <type>transmission_interface/SimpleTransmission</type>
     <joint name="LHip">
-      <hardwareInterface>hardware_interface/PositionJointInterface</hardwareInterface>
+      <hardwareInterface>hardware_interface/VelocityJointInterface</hardwareInterface>
     </joint>
     <actuator name="motorLHip">
-      <hardwareInterface>hardware_interface/PositionJointInterface</hardwareInterface>
+      <hardwareInterface>hardware_interface/VelocityJointInterface</hardwareInterface>
       <mechanicalReduction>1</mechanicalReduction>
     </actuator>
