Commit message: Add files via upload

File: yoyoman01_traject/config/yoyoman01.srdf.xacro (robot description, xacro)
@@ -15,4 +15,68 @@
       <link name="RArmLink" />
       <joint name="fixed" />
+      <joint name="RKnee" />
+      <joint name="LKnee" />
+      <joint name="RFoot" />
+      <joint name="LFoot" />
+      <link name="base_link" />
+      <link name="RKneeLink" />
+      <link name="LKneeLink" />
+      <link name="RFootLink" />
+      <link name="LFootLink" />
    </group>
+   <disable_collisions link1='Rarm' link2='Larm' reason='Never' />
+   <disable_collisions link1='Rarm' link2='RHip' reason='Never' />
+   <disable_collisions link1='Rarm' link2='LHip' reason='Never' />
+   <disable_collisions link1='Rarm' link2='Head' reason='Never' />
+   <disable_collisions link1='Rarm' link2='Neck' reason='Never' />
+   <disable_collisions link1='Rarm' link2='RKnee' reason='Never' />
+   <disable_collisions link1='Rarm' link2='LKnee' reason='Never' />
+   <disable_collisions link1='Rarm' link2='RFoot' reason='Never' />
+   <disable_collisions link1='Rarm' link2='LFoot' reason='Never' />
+   <disable_collisions link1='Rarm' link2='fixed' reason='Never' />
+   <disable_collisions link1='Larm' link2='RHip' reason='Never' />
+   <disable_collisions link1='Larm' link2='LHip' reason='Never' />
+   <disable_collisions link1='Larm' link2='Head' reason='Never' />
+   <disable_collisions link1='Larm' link2='Neck' reason='Never' />
+   <disable_collisions link1='Larm' link2='RKnee' reason='Never' />
+   <disable_collisions link1='Larm' link2='LKnee' reason='Never' />
+   <disable_collisions link1='Larm' link2='RFoot' reason='Never' />
+   <disable_collisions link1='Larm' link2='LFoot' reason='Never' />
+   <disable_collisions link1='Larm' link2='fixed' reason='Never' />
+   <disable_collisions link1='RHip' link2='LHip' reason='Never' />
+   <disable_collisions link1='RHip' link2='Head' reason='Never' />
+   <disable_collisions link1='RHip' link2='Neck' reason='Never' />
+   <disable_collisions link1='RHip' link2='RKnee' reason='Never' />
+   <disable_collisions link1='RHip' link2='LKnee' reason='Never' />
+   <disable_collisions link1='RHip' link2='RFoot' reason='Never' />
+   <disable_collisions link1='RHip' link2='LFoot' reason='Never' />
+   <disable_collisions link1='RHip' link2='fixed' reason='Never' />
+   <disable_collisions link1='LHip' link2='Head' reason='Never' />
+   <disable_collisions link1='LHip' link2='Neck' reason='Never' />
+   <disable_collisions link1='LHip' link2='RKnee' reason='Never' />
+   <disable_collisions link1='LHip' link2='LKnee' reason='Never' />
+   <disable_collisions link1='LHip' link2='RFoot' reason='Never' />
+   <disable_collisions link1='LHip' link2='LFoot' reason='Never' />
+   <disable_collisions link1='LHip' link2='fixed' reason='Never' />
+   <disable_collisions link1='Head' link2='Neck' reason='Never' />
+   <disable_collisions link1='Head' link2='RKnee' reason='Never' />
+   <disable_collisions link1='Head' link2='LKnee' reason='Never' />
+   <disable_collisions link1='Head' link2='RFoot' reason='Never' />
+   <disable_collisions link1='Head' link2='LFoot' reason='Never' />
+   <disable_collisions link1='Head' link2='fixed' reason='Never' />
+   <disable_collisions link1='Neck' link2='RKnee' reason='Never' />
+   <disable_collisions link1='Neck' link2='LKnee' reason='Never' />
+   <disable_collisions link1='Neck' link2='RFoot' reason='Never' />
+   <disable_collisions link1='Neck' link2='LFoot' reason='Never' />
+   <disable_collisions link1='Neck' link2='fixed' reason='Never' />
+   <disable_collisions link1='RKnee' link2='LKnee' reason='Never' />
+   <disable_collisions link1='RKnee' link2='RFoot' reason='Never' />
+   <disable_collisions link1='RKnee' link2='LFoot' reason='Never' />
+   <disable_collisions link1='RKnee' link2='fixed' reason='Never' />
+   <disable_collisions link1='LKnee' link2='RFoot' reason='Never' />
+   <disable_collisions link1='LKnee' link2='LFoot' reason='Never' />
+   <disable_collisions link1='LKnee' link2='fixed' reason='Never' />
+   <disable_collisions link1='RFoot' link2='LFoot' reason='Never' />
+   <disable_collisions link1='RFoot' link2='fixed' reason='Never' />
+   <disable_collisions link1='LFoot' link2='fixed' reason='Never' />
 </robot>

File: yoyoman01_traject/urdf/yoyoman01.xacro (robot description, xacro)
@@ -10,9 +10,9 @@
       <color rgba="0 0 0.8 1"/>
    </material>
-   <!--link name="world"/>
+   <link name="world"/>
   <joint name="fixed" type="fixed">
     <parent link="world"/>
     <child link="base_link"/>
-</joint-->
+</joint>
   <link name="base_link">
     <inertial>
@@ -40,5 +40,5 @@
     <origin rpy="0 0 0" xyz="0 0 0.675"/>
     <axis xyz="0 1 0"/>
-    <limit effort="10.5" lower="-0.5" upper="0.5" velocity="1"/>
+    <limit effort="0.5" lower="0" upper="0.5" velocity="1"/>
   </joint>
   <link name="NeckLink">
@@ -66,5 +66,5 @@
     <origin rpy="0 0 0" xyz="0 0 0.064502"/>
     <axis xyz="0 1 0"/>
-    <limit effort="10.5" lower="-0.5" upper="0.5" velocity="1"/>
+    <limit effort="0.5" lower="0" upper="0.5" velocity="1"/>
   </joint>
   <link name="HeadLink">
@@ -93,5 +93,5 @@
     <origin rpy="0 0 0" xyz="0 -0.155 0.589901 "/>
     <axis xyz="0 1 0"/>
-    <limit effort="50" lower="-3" upper="3" velocity="10"/>
+    <limit effort="5" lower="0" upper="5" velocity="1"/>
   </joint>
 <link name="RArmLink">
@@ -119,5 +119,5 @@
     <origin rpy="0 0 0" xyz="0 0.155 0.589901 "/>
     <axis xyz="0 1 0"/>
-    <limit effort="50" lower="-3" upper="3" velocity="10"/>
+    <limit effort="2.57" lower="-0.349066" upper="0.279253" velocity="1.9"/>
   </joint>
 <link name="LArmLink">
@@ -145,5 +145,5 @@
     <origin rpy="0 0 0" xyz="0 -0.09 0"/>
     <axis xyz="0 1 0"/>
-    <limit effort="600" lower="-3" upper="3" velocity="10"/>
+    <limit effort="6" lower="0" upper="6" velocity="1"/>
   </joint>
   <link name="RHipLink">
@@ -171,5 +171,5 @@
     <origin rpy="0 0 0" xyz="0 0.09 0"/>
     <axis xyz="0 1 0"/>
-    <limit effort="600" lower="-3" upper="3" velocity="10"/>
+    <limit effort="6" lower="0" upper="6" velocity="1"/>
   </joint>
   <link name="LHipLink">

Commit message: removing velocity interface and adding ROS PID for gazebo gravity issue

File: yoyoman01_traject/config/yoyoman01.srdf.xacro (robot description, xacro)
@@ -14,5 +14,5 @@
       <link name="RHipLink" />
       <link name="RArmLink" />
-      <joint name="fixed" />
+      <!--joint name="fixed" /-->
       <joint name="RKnee" />
       <joint name="LKnee" />
@@ -34,5 +34,5 @@
    <disable_collisions link1='Rarm' link2='RFoot' reason='Never' />
    <disable_collisions link1='Rarm' link2='LFoot' reason='Never' />
-   <disable_collisions link1='Rarm' link2='fixed' reason='Never' />
+   <!--disable_collisions link1='Rarm' link2='fixed' reason='Never' /-->
    <disable_collisions link1='Larm' link2='RHip' reason='Never' />
    <disable_collisions link1='Larm' link2='LHip' reason='Never' />
@@ -43,5 +43,5 @@
    <disable_collisions link1='Larm' link2='RFoot' reason='Never' />
    <disable_collisions link1='Larm' link2='LFoot' reason='Never' />
-   <disable_collisions link1='Larm' link2='fixed' reason='Never' />
+   <!--disable_collisions link1='Larm' link2='fixed' reason='Never' /-->
    <disable_collisions link1='RHip' link2='LHip' reason='Never' />
    <disable_collisions link1='RHip' link2='Head' reason='Never' />
@@ -51,5 +51,5 @@
    <disable_collisions link1='RHip' link2='RFoot' reason='Never' />
    <disable_collisions link1='RHip' link2='LFoot' reason='Never' />
-   <disable_collisions link1='RHip' link2='fixed' reason='Never' />
+   <!--disable_collisions link1='RHip' link2='fixed' reason='Never' /-->
    <disable_collisions link1='LHip' link2='Head' reason='Never' />
    <disable_collisions link1='LHip' link2='Neck' reason='Never' />
@@ -58,5 +58,5 @@
    <disable_collisions link1='LHip' link2='RFoot' reason='Never' />
    <disable_collisions link1='LHip' link2='LFoot' reason='Never' />
-   <disable_collisions link1='LHip' link2='fixed' reason='Never' />
+   <!--disable_collisions link1='LHip' link2='fixed' reason='Never' /-->
    <disable_collisions link1='Head' link2='Neck' reason='Never' />
    <disable_collisions link1='Head' link2='RKnee' reason='Never' />
@@ -64,19 +64,19 @@
    <disable_collisions link1='Head' link2='RFoot' reason='Never' />
    <disable_collisions link1='Head' link2='LFoot' reason='Never' />
-   <disable_collisions link1='Head' link2='fixed' reason='Never' />
+   <!--disable_collisions link1='Head' link2='fixed' reason='Never' /-->
    <disable_collisions link1='Neck' link2='RKnee' reason='Never' />
    <disable_collisions link1='Neck' link2='LKnee' reason='Never' />
    <disable_collisions link1='Neck' link2='RFoot' reason='Never' />
    <disable_collisions link1='Neck' link2='LFoot' reason='Never' />
-   <disable_collisions link1='Neck' link2='fixed' reason='Never' />
+   <!--disable_collisions link1='Neck' link2='fixed' reason='Never' /-->
    <disable_collisions link1='RKnee' link2='LKnee' reason='Never' />
    <disable_collisions link1='RKnee' link2='RFoot' reason='Never' />
    <disable_collisions link1='RKnee' link2='LFoot' reason='Never' />
-   <disable_collisions link1='RKnee' link2='fixed' reason='Never' />
+   <!--disable_collisions link1='RKnee' link2='fixed' reason='Never' /-->
    <disable_collisions link1='LKnee' link2='RFoot' reason='Never' />
    <disable_collisions link1='LKnee' link2='LFoot' reason='Never' />
-   <disable_collisions link1='LKnee' link2='fixed' reason='Never' />
+   <!--disable_collisions link1='LKnee' link2='fixed' reason='Never' /-->
    <disable_collisions link1='RFoot' link2='LFoot' reason='Never' />
-   <disable_collisions link1='RFoot' link2='fixed' reason='Never' />
-   <disable_collisions link1='LFoot' link2='fixed' reason='Never' />
+   <!--disable_collisions link1='RFoot' link2='fixed' reason='Never' /-->
+   <!--disable_collisions link1='LFoot' link2='fixed' reason='Never' /-->
 </robot>

File: yoyoman01_traject/urdf/yoyoman01.xacro (robot description, xacro)
@@ -302,8 +302,8 @@
     <type>transmission_interface/SimpleTransmission</type>
     <joint name="Head">
-      <hardwareInterface>hardware_interface/VelocityJointInterface</hardwareInterface>
+      <hardwareInterface>hardware_interface/PositionJointInterface</hardwareInterface>
     </joint>
     <actuator name="motorHead">
-      <hardwareInterface>hardware_interface/VelocityJointInterface</hardwareInterface>
+      <hardwareInterface>hardware_interface/PositionJointInterface</hardwareInterface>
       <mechanicalReduction>1</mechanicalReduction>
     </actuator>
@@ -312,8 +312,8 @@
     <type>transmission_interface/SimpleTransmission</type>
     <joint name="Neck">
-      <hardwareInterface>hardware_interface/VelocityJointInterface</hardwareInterface>
+      <hardwareInterface>hardware_interface/PositionJointInterface</hardwareInterface>
     </joint>
     <actuator name="motorNeck">
-      <hardwareInterface>hardware_interface/VelocityJointInterface</hardwareInterface>
+      <hardwareInterface>hardware_interface/PositionJointInterface</hardwareInterface>
       <mechanicalReduction>1</mechanicalReduction>
     </actuator>
@@ -322,8 +322,8 @@
     <type>transmission_interface/SimpleTransmission</type>
     <joint name="Rarm">
-      <hardwareInterface>hardware_interface/VelocityJointInterface</hardwareInterface>
+      <hardwareInterface>hardware_interface/PositionJointInterface</hardwareInterface>
     </joint>
     <actuator name="motorRarm">
-      <hardwareInterface>hardware_interface/VelocityJointInterface</hardwareInterface>
+      <hardwareInterface>hardware_interface/PositionJointInterface</hardwareInterface>
       <mechanicalReduction>1</mechanicalReduction>
     </actuator>
@@ -332,8 +332,8 @@
     <type>transmission_interface/SimpleTransmission</type>
     <joint name="Larm">
-      <hardwareInterface>hardware_interface/VelocityJointInterface</hardwareInterface>
+      <hardwareInterface>hardware_interface/PositionJointInterface</hardwareInterface>
     </joint>
     <actuator name="motorLarm">
-      <hardwareInterface>hardware_interface/VelocityJointInterface</hardwareInterface>
+      <hardwareInterface>hardware_interface/PositionJointInterface</hardwareInterface>
       <mechanicalReduction>1</mechanicalReduction>
     </actuator>
@@ -342,8 +342,8 @@
     <type>transmission_interface/SimpleTransmission</type>
     <joint name="RHip">
-      <hardwareInterface>hardware_interface/VelocityJointInterface</hardwareInterface>
+      <hardwareInterface>hardware_interface/PositionJointInterface</hardwareInterface>
     </joint>
     <actuator name="motorRHip">
-      <hardwareInterface>hardware_interface/VelocityJointInterface</hardwareInterface>
+      <hardwareInterface>hardware_interface/PositionJointInterface</hardwareInterface>
       <mechanicalReduction>1</mechanicalReduction>
     </actuator>
@@ -352,8 +352,8 @@
     <type>transmission_interface/SimpleTransmission</type>
     <joint name="LHip">
-      <hardwareInterface>hardware_interface/VelocityJointInterface</hardwareInterface>
+      <hardwareInterface>hardware_interface/PositionJointInterface</hardwareInterface>
     </joint>
     <actuator name="motorLHip">
-      <hardwareInterface>hardware_interface/VelocityJointInterface</hardwareInterface>
+      <hardwareInterface>hardware_interface/PositionJointInterface</hardwareInterface>
       <mechanicalReduction>1</mechanicalReduction>
     </actuator>
